Commit message: new updates - static map, robot camera, etc.

File: sim_robot/camera/urdf/rear_camera_support.urdf.xacro (robot description, xacro)
@@ -36,5 +36,6 @@
             <parent link="${main_camera_base}"/>
             <child link="${prefix}camera_support"/>
-            <origin xyz="-${0.075-width/2} 0 0.8" rpy="0 0 3.14"/>
+            <!-- <origin xyz="-${0.075-width/2} 0 0.8" rpy="0 0 3.14"/> -->
+            <origin xyz="${0.075-width/2} 0.0 0.8" rpy="0 1.0 0"/> <!-- for downward-facing configuration-->
             <axis xyz="0 0 1"/>
         </joint>
