Commit message: Update freight.urdf.xacro

File: sim_robot/base/urdf/freight.urdf.xacro (robot description, xacro)
@@ -16,5 +16,5 @@
       <origin rpy="0 0 0" xyz="0 0 0" />
       <geometry>
-        <mesh filename="package://freight_description/base/meshes/base_link.dae" />
+        <mesh filename="package://sim_robot/base/meshes/base_link.dae" />
       </geometry>
       <material name="">
@@ -25,5 +25,5 @@
       <origin rpy="0 0 0" xyz="0 0 0" />
       <geometry>
-        <mesh filename="package://freight_description/base/meshes/base_link_collision.STL" />
+        <mesh filename="package://sim_robot/base/meshes/base_link_collision.STL" />
       </geometry>
     </collision>
@@ -38,5 +38,5 @@
       <origin rpy="0 0 0" xyz="0 0 0" />
       <geometry>
-        <mesh filename="package://freight_description/base/meshes/r_wheel_link.STL" />
+        <mesh filename="package://sim_robot/base/meshes/r_wheel_link.STL" />
       </geometry>
       <material name="">
@@ -47,5 +47,5 @@
       <origin rpy="0 0 0" xyz="0 0 0" />
       <geometry>
-        <mesh filename="package://freight_description/base/meshes/r_wheel_link_collision.STL" />
+        <mesh filename="package://sim_robot/base/meshes/r_wheel_link_collision.STL" />
       </geometry>
     </collision>
@@ -68,5 +68,5 @@
       <origin rpy="0 0 0" xyz="0 0 0" />
       <geometry>
-        <mesh filename="package://freight_description/base/meshes/l_wheel_link.STL" />
+        <mesh filename="package://sim_robot/base/meshes/l_wheel_link.STL" />
       </geometry>
       <material name="">
@@ -77,5 +77,5 @@
       <origin rpy="0 0 0" xyz="0 0 0" />
       <geometry>
-        <mesh filename="package://freight_description/base/meshes/l_wheel_link_collision.STL" />
+        <mesh filename="package://sim_robot/base/meshes/l_wheel_link_collision.STL" />
       </geometry>
     </collision>
@@ -98,5 +98,5 @@
       <origin rpy="0 0 0" xyz="0 0 0" />
       <geometry>
-        <mesh filename="package://freight_description/base/meshes/estop_link.STL" />
+        <mesh filename="package://sim_robot/base/meshes/estop_link.STL" />
       </geometry>
       <material name="">
@@ -107,5 +107,5 @@
       <origin rpy="0 0 0" xyz="0 0 0" />
       <geometry>
-        <mesh filename="package://freight_description/base/meshes/estop_link.STL" />
+        <mesh filename="package://sim_robot/base/meshes/estop_link.STL" />
       </geometry>
     </collision>
@@ -127,5 +127,5 @@
       <origin rpy="0 0 0" xyz="0 0 0" />
       <geometry>
-        <mesh filename="package://freight_description/base/meshes/laser_link.STL" />
+        <mesh filename="package://sim_robot/base/meshes/laser_link.STL" />
       </geometry>
       <material name="">
@@ -136,5 +136,5 @@
       <origin rpy="0 0 0" xyz="0 0 0" />
       <geometry>
-        <mesh filename="package://freight_description/base/meshes/laser_link.STL" />
+        <mesh filename="package://sim_robot/base/meshes/laser_link.STL" />
       </geometry>
     </collision>
